File: Hardware/Current_Sense_Nano/Current_Sense_Nano.sch (KiCad schematic (older format))
At the start: 7 parts, among them J1 Conn_01x06, SW1 SW_DP3T, U1 INA214AIDCKR

Commit message: v01 layout complete
Parts:
- added H1, H2: MountingHole, MountingHole:MountingHole_3.2mm_M3, symbol Mechanical:MountingHole
- added J2, J3, J4, J5, J6: Conn_01x01, Current_Sense_Nano:z_BBC-BIT, symbol Connector_Generic:Conn_01x01
- added JP1: SolderJumper_2_Bridged, Jumper:SolderJumper-2_P1.3mm_Bridged_RoundedPad1.0x1.5mm, symbol Jumper:SolderJumper_2_Bridged
- C1: footprint (none) -> Capacitor_SMD:C_0603_1608Metric
- J1: footprint (none) -> Current_Sense_Nano:PinHeader_1x06_P2.54mm_Vertical_NoSilk
- R1, R2, R3: footprint (none) -> Resistor_SMD:R_0805_2012Metric
- SW1: footprint (none) -> Current_Sense_Nano:Switch_Slide_20.7x10.4mm_G-128S-0157
- U1: footprint DCK6 -> footprints:INA214AIDCKR
Connections:
- net pos_mA: now reaches SW1.1
- net pos_mA: now also R1.2, R2.1, SW1.5
- net IN-: now reaches SW1.2
- net IN-: now also J1.2 (Pin_2), R3.2, SW1.6, U1.5 (IN-), J3.1 (Pin_1)
- net pos_uA: now reaches SW1.3
- net pos_uA: now also R2.2, R3.1, SW1.7
- net REF: now reaches U1.1 (REF)
- net REF: now also J1.6 (Pin_6), JP1.1 (A)
- net GND: now reaches U1.2 (GND)
- net GND: now also C1.2, J1.4 (Pin_4), J5.1 (Pin_1), JP1.2 (B)
- net VS: now reaches U1.3 (V+)
- net VS: now also C1.1, J1.3 (Pin_3), J4.1 (Pin_1)
- net IN+: now reaches U1.4 (IN+)
- net IN+: now also J1.1 (Pin_1), R1.1, J2.1 (Pin_1)
- net OUT: now reaches U1.6 (OUT)
- net OUT: now also J1.5 (Pin_5), J6.1 (Pin_1)
Other:
- note added: "Cut to use\nseparate refernce\nvoltage"
- moved on the sheet: C1, J1, R1, R2, R3, SW1, U1
